Commit message: Add attachement plate between sensor and robot

File: urdf/brace_top_setup.urdf (robot description, URDF)
Before this commit: robot brace_top_setup, 3 links, 2 joints
Links:
- link base_link: mass 0.022610061223038 -> 0.0667407034097946
Joints:
- joint Joint1: origin xyz=0 0 -0.390748 rpy=0 0 0 -> xyz=0 0 -0.0249999999999998 rpy=0 0 0
- joint Joint2: origin xyz=0 0 0.362 rpy=0 0 0 -> xyz=0 0 -0.377748 rpy=0 0 0

Commit message: [23-02-16] [modification urdf and inertia]

File: urdf/brace_top_setup.urdf (robot description, URDF)
Before this commit: robot brace_top_setup, 3 links, 2 joints
Links:
- link Link1: mass 0.018528460193251 -> 0.09563; geometry collision mesh filename=package://brace_top_setup2/meshes/Link1.STL; visual mesh filename=package://brace_top_setup2/meshes/Link1.STL
- link Link2: mass 1.16495586721261 -> 1.598; geometry collision mesh filename=package://brace_top_setup2/meshes/Link2.STL; visual mesh filename=package://brace_top_setup2/meshes/Link2.STL
- link base_link: mass 0.0667407034097946 -> 0.37798; geometry collision mesh filename=package://brace_top_setup2/meshes/base_link.STL; visual mesh filename=package://brace_top_setup2/meshes/base_link.STL
Joints:
- joint Joint1: origin xyz=0 0 -0.0249999999999998 rpy=0 0 0 -> xyz=0 0 -0.402748 rpy=0 0 0
- joint Joint2: origin xyz=0 0 -0.377748 rpy=0 0 0 -> xyz=0 0 0.362 rpy=0 0 0

Commit message: [new modification to repair error in link names]

File: urdf/brace_top_setup.urdf (robot description, URDF)
Before this commit: robot brace_top_setup2, 3 links, 2 joints
Links:
- link Link1: mass 0.09563 -> 0.144521989507358; geometry collision mesh filename=package://brace_top_setup/meshes/Link1.STL; visual mesh filename=package://brace_top_setup/meshes/Link1.STL
- link Link2: mass 1.598 -> 1.55948160838922; geometry collision mesh filename=package://brace_top_setup/meshes/Link2.STL; visual mesh filename=package://brace_top_setup/meshes/Link2.STL
- link base_link: mass 0.37798 -> 0.48452022632218; geometry collision mesh filename=package://brace_top_setup/meshes/base_link.STL; visual mesh filename=package://brace_top_setup/meshes/base_link.STL

Commit message: [modification coordinate system link 2 top setup]

File: urdf/brace_top_setup.urdf (robot description, URDF)
Before this commit: robot brace_top_setup, 3 links, 2 joints
Joints:
- joint Joint1: origin xyz=0 0 -0.402748 rpy=0 0 0 -> xyz=0 0 -0.0250000000000002 rpy=0 0 0
- joint Joint2: origin xyz=0 0 0.362 rpy=0 0 0 -> xyz=0 0 -0.377748 rpy=0 0 0

Commit message: modification of the positionning of the thigh and of the inertia

File: urdf/brace_top_setup.urdf (robot description, URDF)
Before this commit: robot brace_top_setup, 3 links, 2 joints
Links:
- link Link1: mass 0.144521989507358 -> 0.09563
- link Link2: mass 1.55948160838922 -> 1.61915
- link base_link: mass 0.48452022632218 -> 0.37798
Joints:
- joint Joint1: origin xyz=0 0 -0.0250000000000002 rpy=0 0 0 -> xyz=0 0 -0.025 rpy=0 0 0
- joint Joint2: origin xyz=0 0 -0.377748 rpy=0 0 0 -> xyz=0 0 -0.365748000000057 rpy=0 0 0

Commit message: modification base link coordinate system brace top setup

File: urdf/brace_top_setup.urdf (robot description, URDF)
Before this commit: robot brace_top_setup, 3 links, 2 joints
Links:
- link Link1: mass 0.09563 -> 0.144521976607445
- link Link2: mass 1.61915 -> 1.56069403714808
- link base_link: mass 0.37798 -> 0.484520226346476
Joints:
- joint Joint1: origin xyz=0 0 -0.025 rpy=0 0 0 -> xyz=0 0 0.0249999999998006 rpy=-3.14159265358979 0 -0.523598775598296

Commit message: new urdf with new cut plane of the femur + brace

File: urdf/brace_top_setup.urdf (robot description, URDF)
Before this commit: robot brace_top_setup, 3 links, 2 joints
Links:
- link Link2: mass 1.56069403714808 -> 2.2612238536076
- link base_link: mass 0.484520226346476 -> 0.386438799959444
Joints:
- joint Joint1: origin xyz=0 0 0.0249999999998006 rpy=-3.14159265358979 0 -0.523598775598296 -> xyz=0 0 -0.025 rpy=0 0 0
- joint Joint2: origin xyz=0 0 -0.365748000000057 rpy=0 0 0 -> xyz=0 0 -0.365747999999879 rpy=0 0 0

Commit message: try of a new urdf with stl files that are not empty

File: urdf/brace_top_setup.urdf (robot description, URDF)
Before this commit: robot brace_top_setup, 3 links, 2 joints
Links:
- link Link1: mass 0.144521976607445 -> 0.1445219727359
- link Link2: mass 2.2612238536076 -> 2.25336370362878
- link base_link: mass 0.386438799959444 -> 0.475317681721771
Joints:
- joint Joint2: origin xyz=0 0 -0.365747999999879 rpy=0 0 0 -> xyz=0 0 -0.365748 rpy=0 0 0

Commit message: changing the reference coordinate system for base_link to align the X with the screws axis

File: urdf/brace_top_setup.urdf (robot description, URDF)
Before this commit: robot brace_top_setup, 3 links, 2 joints
Links:
- link Link2: mass 2.25336370362878 -> 2.25336370362882
Joints:
- joint Joint1: origin xyz=0 0 -0.025 rpy=0 0 0 -> xyz=0 0 -0.025 rpy=0 0 -2.61799387799149

Commit message: changing the sense of the axis

File: urdf/brace_top_setup.urdf (robot description, URDF)
Before this commit: robot brace_top_setup, 3 links, 2 joints
Joints:
- joint Joint1: origin xyz=0 0 -0.025 rpy=0 0 -2.61799387799149 -> xyz=0 0 -0.025 rpy=0 0 0.523598775598301

Commit message: new inertia corresponding to reality

File: urdf/brace_top_setup.urdf (robot description, URDF)
Before this commit: robot brace_top_setup, 3 links, 2 joints
Links:
- link Link1: mass 0.1445219727359 -> 0.09563
- link Link2: mass 2.25336370362882 -> 2.47015
- link base_link: mass 0.475317681721771 -> 0.37798

Commit message: urdf without the brace : be careful, the inertia are not the good ones

File: urdf/brace_top_setup.urdf (robot description, URDF)
Before this commit: robot brace_top_setup, 3 links, 2 joints
Links:
- link Link1: mass 0.09563 -> 0.144521976607445
- link Link2: mass 2.47015 -> 1.56069403714808
- link base_link: mass 0.37798 -> 0.386438799959442
Joints:
- joint Joint1: origin xyz=0 0 -0.025 rpy=0 0 0.523598775598301 -> xyz=0 0 -0.025 rpy=0 0 0

Commit message: changing the part under the femur (to fit the new cones calib part)

File: urdf/brace_top_setup.urdf (robot description, URDF)
Before this commit: robot brace_top_setup_brace, 3 links, 2 joints
Links:
- link Link2: mass 1.56069403714808 -> 1.72264558496205
- link base_link: mass 0.386438799959442 -> 0.386438799959444
Joints:
- joint Joint2: origin xyz=0 0 -0.365748 rpy=0 0 0 -> xyz=-0.000349804795560293 0.000497472935857356 -0.385747999999876 rpy=0 0 -0.0176473497580653

Commit message: changing the part under the femur to adapt to the new calib part (with cones)

File: urdf/brace_top_setup.urdf (robot description, URDF)
Before this commit: robot brace_top_setup, 3 links, 2 joints
Links:
- link Link1: mass 0.144521976607445 -> 0.144522029461181
- link Link2: mass 1.72264558496205 -> 1.72261543966663
- link base_link: mass 0.386438799959444 -> 0.38643879994659
Joints:
- joint Joint2: origin xyz=-0.000349804795560293 0.000497472935857356 -0.385747999999876 rpy=0 0 -0.0176473497580653 -> xyz=0 0 -0.385747999999999 rpy=0 0 0

Commit message: changing the position of the thigh on the setup to fit reality

File: urdf/brace_top_setup.urdf (robot description, URDF)
Before this commit: robot brace_top_setup, 3 links, 2 joints
Links:
- link Link1: mass 0.144522029461181 -> 0.144521976607445
- link Link2: mass 1.72261543966663 -> 1.72264634502229
- link base_link: mass 0.38643879994659 -> 0.386438799959442

Commit message: changing the plate under the femur to replace it by the previous one that is smaller

File: urdf/brace_top_setup.urdf (robot description, URDF)
Before this commit: robot brace_top_setup, 3 links, 2 joints
Links:
- link Link2: mass 1.72264634502229 -> 1.72264634502227

Commit message: changing the axis for base_link to fit the axis of panda_link8

File: urdf/brace_top_setup.urdf (robot description, URDF)
Before this commit: robot brace_top_setup, 3 links, 2 joints
Joints:
- joint Joint1: origin xyz=0 0 -0.025 rpy=0 0 0 -> xyz=0 0 0.025 rpy=3.14159265358979 0 0

Commit message: replacing some 3d printed parts by machined ones

File: urdf/brace_top_setup.urdf (robot description, URDF)
Before this commit: robot brace_top_setup, 3 links, 2 joints
Links:
- link Link1: mass 0.144521976607445 -> 0.144522012260847
- link Link2: mass 1.72264634502227 -> 1.86856414903318
- link base_link: mass 0.386438799959442 -> 0.510468252967356
Joints:
- joint Joint1: origin xyz=0 0 0.025 rpy=3.14159265358979 0 0 -> xyz=0 0 0.02565 rpy=-3.14159265358979 0 0
- joint Joint2: origin xyz=0 0 -0.385747999999999 rpy=0 0 0 -> xyz=0 0 -0.377748 rpy=0 0 0

Commit message: correcting an error of coaxiality between 2 parts

File: urdf/brace_top_setup.urdf (robot description, URDF)
Before this commit: robot brace_top_setup, 3 links, 2 joints
Links:
- link Link2: mass 1.86856414903318 -> 1.86856414903311
- link base_link: mass 0.510468252967356 -> 0.510468252967497
Joints:
- joint Joint2: origin xyz=0 0 -0.377748 rpy=0 0 0 -> xyz=0 0 -0.377748000000005 rpy=0 0 0

Commit message: changing the definition of base link cs

File: urdf/brace_top_setup.urdf (robot description, URDF)
Before this commit: robot brace_top_setup, 3 links, 2 joints
Links:
- link Link1: mass 0.144522012260847 -> 0.144522012260846
- link Link2: mass 1.86856414903311 -> 1.86856414903305
- link base_link: mass 0.510468252967497 -> 0.510468252968612
Joints:
- joint Joint1: origin xyz=0 0 0.02565 rpy=-3.14159265358979 0 0 -> xyz=0 0 0.02565 rpy=3.14159265358979 0 0
- joint Joint2: origin xyz=0 0 -0.377748000000005 rpy=0 0 0 -> xyz=0 0 -0.377748000000006 rpy=0 0 0

Commit message: correcting errors

File: urdf/brace_top_setup.urdf (robot description, URDF)
Before this commit: robot brace_top_setup, 3 links, 2 joints
Links:
- link Link1: mass 0.144522012260847 -> 0.144521976607446
- link Link2: mass 1.86856414903318 -> 1.86856831514572
Joints:
- joint Joint1: origin xyz=0 0 0.02565 rpy=-3.14159265358979 0 0 -> xyz=0 0 0.0256500000001189 rpy=-3.14159265358979 0 0
- joint Joint2: origin xyz=0 0 -0.377748 rpy=0 0 0 -> xyz=0 0 -0.377747999999882 rpy=0 0 0

Commit message: correcting errors in Link2

File: urdf/brace_top_setup.urdf (robot description, URDF)
Before this commit: robot brace_top_setup, 3 links, 2 joints
Links:
- link Link2: mass 1.86856414903305 -> 1.62403649405776
Joints:
- joint Joint1: origin xyz=0 0 0.02565 rpy=3.14159265358979 0 0 -> xyz=-0.19887040656027 0.0129955434612824 0.11187805288069 rpy=1.57079632679489 0.296705972839033 0
- joint Joint2: origin xyz=0 0 -0.377748000000006 rpy=0 0 0 -> xyz=0 0 -0.377748 rpy=0 0 0

Commit message: correct an error in origin of baselink

File: urdf/brace_top_setup.urdf (robot description, URDF)
Before this commit: robot brace_top_setup, 3 links, 2 joints
Joints:
- joint Joint1: origin xyz=-0.19887040656027 0.0129955434612824 0.11187805288069 rpy=1.57079632679489 0.296705972839033 0 -> xyz=0 0 0.02565 rpy=3.14159265358979 0 0

Commit message: verif

File: urdf/brace_top_setup.urdf (robot description, URDF)
Before this commit: robot brace_top_setup, 3 links, 2 joints
Links:
- link Link1: mass 0.144522012260846 -> 0.144521976607445
- link Link2: mass 1.62403649405776 -> 1.62404066017064
- link base_link: mass 0.510468252968612 -> 0.510468252967356
Joints:
- joint Joint1: origin xyz=0 0 0.02565 rpy=3.14159265358979 0 0 -> xyz=0 0 0.0256499999999998 rpy=-3.14159265358979 0 0

Commit message: modif of Link2 origin to be on the upper side of femur plate and not lower side

File: urdf/brace_top_setup.urdf (robot description, URDF)
Before this commit: robot brace_top_setup, 3 links, 2 joints
Joints:
- joint Joint2: origin xyz=0 0 -0.377748 rpy=0 0 0 -> xyz=0 0 -0.365748 rpy=0 0 0

Commit message: modif of origin link2

File: urdf/brace_top_setup.urdf (robot description, URDF)
Before this commit: robot brace_top_setup, 3 links, 2 joints
Joints:
- joint Joint1: origin xyz=0 0 0.0256499999999998 rpy=-3.14159265358979 0 0 -> xyz=0 0 0.0256500000000002 rpy=-3.14159265358979 0 0
- joint Joint2: origin xyz=0 0 -0.365748 rpy=0 0 0 -> xyz=0 0 -0.377748 rpy=0 0 0
